File: display_controller/display_controller.kicad_sch (KiCad schematic)
At the start: 2 parts, among them J1 CF314, U1 LVDS391

Commit message: update footprints
Parts:
- J1: footprint (none) -> custom:CF3103S_40pin
- U1: footprint (none) -> custom:PW16
Connections:
- net at J1.11 (RXIN1-): now also U1.14 (2Y); no longer U1. (Vcc)
- net at J1.12 (RXIN1+): now also U1.13 (2Z); no longer U1. (Vcc)
- net at J1.14 (RXIN2-): now also U1.12 (3Y); no longer U1. (Vcc)
- net at J1.15 (RXIN2+): now also U1.11 (3Z); no longer U1. (Vcc)
- net at J1.17 (RXCLKIN-): now also U1.10 (4Y); no longer U1. (Vcc)
- net at J1.18 (RXCLKIN+): now also U1.9 (4Z); no longer U1. (Vcc)
- net at J1.8 (RXIN0-): now also U1.16 (1Y); no longer U1. (Vcc)
- net at J1.9 (RXIN0+): now also U1.15 (1Z); no longer U1. (Vcc)
Changed lines of the file:
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@@
       (effects (font (size 1.27 1.27)))
     )
-    (property "Footprint" "" (at 206.756 65.786 0)
+    (property "Footprint" "custom:PW16" (at 206.756 65.786 0)
       (effects (font (size 1.27 1.27)) hide)
     )
-    (property "Datasheet" "${KIPRJMOD}/datasheets/LVDS391.pdf" (at 206.756 65.786 0)
+    (property "Datasheet" "https://www.ti.com/lit/ds/symlink/sn65lvds387.pdf?ts=1704479809106&ref_url=https%253A%252F%252Fwww.mouser.com%252F" (at 206.756 65.786 0)
       (effects (font (size 1.27 1.27)) hide)
     )
-    (pin "")
-    (pin "")
-    (pin "")
-    (pin "")
-    (pin "")
-    (pin "")
-    (pin "")
-    (pin "")
-    (pin "")
-    (pin "")
-    (pin "")
-    (pin "")
-    (pin "")
-    (pin "")
-    (pin "")
-    (pin "")
+    (pin "1")
+    (pin "10")
+    (pin "11")
+    (pin "12")
+    (pin "13")
+    (pin "14")
+    (pin "15")
+    (pin "16")
+    (pin "2")
+    (pin "3")
+    (pin "4")
+    (pin "5")
+    (pin "6")
+    (pin "7")
+    (pin "8")
+    (pin "9")
     (instances
       (project "display_controller"
@@
       (effects (font (size 1.27 1.27)) (justify left))
     )
-    (property "Footprint" "" (at 251.206 89.916 0)
+    (property "Footprint" "custom:CF3103S_40pin" (at 251.206 89.916 0)
       (effects (font (size 1.27 1.27)) hide)
     )

Commit message: change FPC connector
Parts:
- J1: value CF314 -> FPC CONN; footprint custom:CF3103S_40pin -> custom:CONN_4-1734592-0_TYCO
Changed lines of the file:
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@@
       (effects (font (size 1.27 1.27)) (justify left))
     )
-    (property "Value" "CF314" (at 253.746 93.091 0)
+    (property "Value" "FPC CONN" (at 253.746 93.091 0)
       (effects (font (size 1.27 1.27)) (justify left))
     )
-    (property "Footprint" "custom:CF3103S_40pin" (at 251.206 89.916 0)
+    (property "Footprint" "custom:CONN_4-1734592-0_TYCO" (at 251.206 89.916 0)
       (effects (font (size 1.27 1.27)) hide)
     )

Commit message: Add flash modules, MCU, and usb-c receptacle
Parts:
- added J2: USB4105GFA120, custom:GCT_USB4105GFA120, symbol custom:USB4105GFA120
- added U10, U3, U4, U5, U6, U7, U8, U9: GD25Q16, custom:SOP8 150mil, symbol custom:GD25Q16
- added U2: STM32F412RETx, Package_QFP:LQFP-64_10x10mm_P0.5mm, symbol MCU_ST_STM32F4:STM32F412RETx
Connections:
- net GND: now also J1.36 (CABCEN1), J1.37 (CABCEN0), J2.A1_B12 (GND), J2.B1_A12 (GND__1), J2.SH1 (SHELL_GND), J2.SH2 (SHELL_GND__1), J2.SH3 (SHELL_GND__2), J2.SH4 (SHELL_GND__3)
- new net: U2.18 (VSS), U2.31 (VSS), U2.47 (VSS), U2.63 (VSS)
Other:
- note added: "NC"
